File: usdx_mono_PA/usdx_mono_PA.kicad_pcb (KiCad board)
At the start: 2 copper layers, 99.5 x 36.5 mm, 53 parts, among them J1 Conn_01x04, J2 Conn_01x01, J3 Conn_01x04, J5 Conn_01x02, K1 IM01, K2 IM01, Q1 2SC1969, Q2 DTC114EE, Q3 DTC114EE, U1 L7805CDT-TR

Commit message: add mods
Parts:
- moved D1 7.98 mm to (44.7, 53.8), turned to -90 degrees
- moved RV1 7.12 mm to (41.4, 58.7)
- moved L1 4.32 mm to (58.4, 59.2)
- moved L3 4.17 mm to (42.7, 28.7), turned to 0 degrees
- moved C1 4.15 mm to (62.2, 58.2), turned to -90 degrees
- moved R4 4.09 mm to (44.5, 58.6)
- moved C2 3.84 mm to (46.7, 58.7)
- moved C5 3.81 mm to (41.4, 50.3)
- moved C9 2.81 mm to (79.0, 30.0), turned to -90 degrees
- moved R3 2.05 mm to (67.5, 58.7)
- moved C10 1.46 mm to (108.7, 33.5), turned to 180 degrees
- moved R6 1.27 mm to (49.8, 39.9)
- moved R5 1.27 mm to (49.8, 41.9)
- moved L5 1.18 mm to (113.1, 39.4)
- moved C4 1.07 mm to (51.8, 32.0), turned to 90 degrees
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Routing:
- net Net-(C1-Pad1): track 12.6 -> 7.18 mm
- net Net-(Q1-Pad1): track 8.23 -> 5.18 mm
- net Net-(C8-Pad1): track 40.2 -> 38.8 mm
- net rf-r-in: track 23.0 -> 21.7 mm
- net Net-(L2-Pad2): track 26.2 -> 25.0 mm
- net +12V: track 8.52 -> 9.57 mm
- net Net-(C1-Pad2): track 2.84 -> 3.82 mm
- net Net-(C10-Pad1): track 11.3 -> 10.3 mm
- net Net-(L1-Pad2): track 31.0 -> 32.0 mm
- net Net-(C2-Pad2): track 16.3 -> 17.2 mm
- net Net-(C3-Pad2): track 16.2 -> 15.6 mm
- net VCC_PA_B: track 116.7 -> 116.3 mm, vias 3 -> 2
- net RD_B: track 28.7 -> 29.0 mm, vias 0 -> 1

Commit message: add mods on pcb
Routing:
- net GND: track 0.00 -> 0.91 mm, vias 0 -> 211
- net ANT_B: track 21.5 -> 20.8 mm
Other:
- board text added: "F4HTB 2022"

Commit message: add mods
Parts:
- added C19: 100n, Capacitor_SMD:C_0805_2012Metric_Pad1.18x1.45mm_HandSolder, B.Cu at (34.8, 47.6)
- added D4: LED, LED_SMD:LED_0805_2012Metric_Pad1.15x1.40mm_HandSolder, F.Cu at (49.3, 59.4)
- added R10: 420, Resistor_SMD:R_0805_2012Metric_Pad1.20x1.40mm_HandSolder, F.Cu at (45.5, 59.4)
- moved L1 12.1 mm to (60.6, 47.2)
- moved C2 11.3 mm to (49.4, 47.6), turned to 0 degrees
- moved C1 10.9 mm to (63.6, 47.3), turned to 90 degrees
- moved R2 7.12 mm to (69.0, 47.4)
- moved R5 6.86 mm to (49.5, 35.1)
- moved R6 6.23 mm to (49.5, 33.7)
- moved R4 5.87 mm to (45.5, 52.8), turned to 0 degrees
- moved R3 5.46 mm to (69.2, 53.5), turned to 90 degrees
- moved C5 3.47 mm to (39.7, 47.2)
- moved D1 2.06 mm to (46.3, 55.1), turned to 180 degrees
- moved C4 1.80 mm to (53.6, 32.3)
- moved R1 1.42 mm to (73.7, 53.5)
- moved C15 0.38 mm to (85.0, 51.0)
- moved Q1 0.09 mm to (46.2, 40.1)
Connections:
- Q1 pad 1: Net-(Q1-Pad1) -> Net-(L1-Pad2)
- Q1 pad 3: Net-(L1-Pad2) -> Net-(Q1-Pad3)
- R5 pad 2: Net-(Q1-Pad1) -> Net-(Q1-Pad3)
- R6 pad 2: Net-(Q1-Pad1) -> Net-(Q1-Pad3)
Routing:
- net Net-(L1-Pad2): track 32.0 -> 16.5 mm
- net +5V: track 95.1 -> 100.9 mm, vias 1 -> 2
- net Net-(Q1-Pad1): track 5.18 -> 0.00 mm
- net Net-(Q1-Pad3): track 0.00 -> 4.56 mm
- net GND: track 0.91 -> 5.05 mm, vias 211 -> 356
- net rf-tx-in: track 36.5 -> 32.6 mm
- net VCC_PA_A: track 6.01 -> 9.61 mm
- net Net-(L2-Pad2): track 25.0 -> 27.7 mm
- net VCC_PA_B: track 116.3 -> 114.1 mm
- net Net-(D4-Pad2): track 0.00 -> 1.81 mm
- net Net-(C2-Pad2): track 17.2 -> 18.3 mm
- net Net-(D3-Pad2): track 2.84 -> 1.95 mm
- net Net-(D2-Pad1): track 4.70 -> 4.03 mm
- net rf-tx-out: track 10.4 -> 9.80 mm

Commit message: add mods
Parts:
- added C20: 470uF, Capacitor_SMD:C_0805_2012Metric_Pad1.18x1.45mm_HandSolder, B.Cu at (113.0, 59.6)
- added J4: Conn_01x02, Jumper:SolderJumper-2_P1.3mm_Open_RoundedPad1.0x1.5mm, B.Cu at (38.3, 30.4)
- D1: footprint Diode_SMD:D_MiniMELF -> Diode_SMD:D_MiniMELF_Handsoldering
- D2, D3: footprint Diode_SMD:D_MiniMELF_Handsoldering -> Diode_SMD:D_MiniMELF
- J1, J3: moved to B.Cu
- Q2, Q3: footprint Package_TO_SOT_SMD:SOT-416 -> Custom:DTC114EE
- moved C4 17.5 mm to (36.7, 27.7), turned to 0 degrees
- moved R4 2.38 mm to (44.8, 50.5), turned to -90 degrees
- moved R6 2.12 mm to (51.7, 33.8), turned to -90 degrees
- moved D1 1.98 mm to (47.3, 53.4), turned to 90 degrees
- moved R5 1.29 mm to (49.6, 33.8), turned to -90 degrees
- moved J5 1.27 mm to (102.6, 59.7), turned to -90 degrees
- moved Q2 1.06 mm to (86.0, 58.4)
- moved R7 0.97 mm to (97.4, 58.5)
- moved C2 0.75 mm to (50.0, 47.3), turned to -90 degrees
- moved Q3 0.52 mm to (106.9, 53.3)
- moved D2 0.31 mm to (91.3, 58.4)
- moved D3 0.09 mm to (109.7, 55.5)
- turned J1 to 0 degrees
- turned J3 to 0 degrees
Connections:
- C4 pad 2: VCC_PA_B -> Net-(C4-Pad2)
- L3 pad 1: VCC_PA_B -> Net-(C4-Pad2)
Routing:
- net Net-(C4-Pad2): track 0.00 -> 8.89 mm
- net PTT: track 30.9 -> 25.5 mm
- net GND: track 5.05 -> 1.16 mm, vias 356 -> 362
- net VCC_PA_B: track 114.1 -> 116.2 mm
- net VCC_PA_A: track 9.61 -> 11.6 mm
- net +5V: track 100.9 -> 102.5 mm
- net Net-(L1-Pad2): track 16.5 -> 15.5 mm
- net Net-(C2-Pad2): track 18.3 -> 19.1 mm
- net Net-(D3-Pad2): track 1.95 -> 2.76 mm
- net Net-(Q1-Pad3): track 4.56 -> 5.21 mm
- net Net-(D3-Pad1): track 3.56 -> 4.20 mm

Commit message: add mods
Parts:
- moved J4 3.42 mm to (39.9, 27.3), turned to 0 degrees
- moved C4 3.35 mm to (39.3, 29.7)
- moved C19 3.03 mm to (33.9, 50.5), turned to 90 degrees
- moved C15 0.87 mm to (84.1, 50.9), turned to 180 degrees
- moved D1 0.86 mm to (47.3, 52.6)
- moved C5 0.51 mm to (40.2, 47.2)
- moved R4 0.38 mm to (44.5, 50.5)
- moved R5 0.13 mm to (49.6, 33.9)
- moved R6 0.13 mm to (51.7, 33.9)
Connections:
- C4 pad 2: Net-(C4-Pad2) -> VCC_PA_B
- J4 pad 2: Net-(C4-Pad2) -> Net-(J4-Pad2)
- L3 pad 1: Net-(C4-Pad2) -> Net-(J4-Pad2)
Routing:
- net Net-(C4-Pad2): track 8.89 -> 0.00 mm
- net Net-(J4-Pad2): track 0.00 -> 3.59 mm
- net VCC_PA_B: track 116.2 -> 118.1 mm
- net RD_B: track 28.9 -> 27.1 mm
- net Net-(C3-Pad2): track 15.6 -> 16.4 mm
- net GND: vias 362 -> 368

Commit message: add mods
Parts:
- C6: footprint Capacitor_SMD:C_0805_2012Metric_Pad1.18x1.45mm_HandSolder -> Capacitor_SMD:C_0402_1005Metric
- R7, R8: value 43 -> 220
- moved C6 4.62 mm to (119.2, 60.3), turned to 180 degrees
- moved C20 0.89 mm to (113.0, 58.7)
- moved R8 0.51 mm to (105.9, 57.7)
Connections:
- R7 pad 1: +5V -> VCC_PA_A
- R8 pad 1: +5V -> VCC_PA_A
Routing:
- net +5V: track 102.5 -> 17.3 mm
- net VCC_PA_A: track 11.6 -> 32.5 mm
- net GND: track 1.16 -> 0.25 mm
- net Net-(J4-Pad2): track 3.59 -> 2.73 mm
- net Net-(D3-Pad1): track 4.20 -> 3.35 mm
