File: usdx_mono_PA/usdx_mono_PA.kicad_sch (KiCad schematic)
At the start: 53 parts, among them J1 Conn_01x04, J2 Conn_01x01, J3 Conn_01x04, J5 Conn_01x02, K1 IM01, K2 IM01, Q1 2SC1969, Q2 DTC114EE, Q3 DTC114EE, U1 L7805CDT-TR

Commit message: add mods
Parts:
- removed Q1: 2SC1969, Package_TO_SOT_THT:TO-220-3_Horizontal_TabDown, symbol Transistor_BJT:2SC1941
- added C19: 100n, Capacitor_SMD:C_0805_2012Metric_Pad1.18x1.45mm_HandSolder, symbol Device:C
- added D4: LED, LED_SMD:LED_0805_2012Metric_Pad1.15x1.40mm_HandSolder, symbol Device:LED
- added Q1: 2SC1969, Package_TO_SOT_THT:TO-220-3_Horizontal_TabDown, symbol Transistor_BJT:2SD1047
- added R10: 420, Resistor_SMD:R_0805_2012Metric_Pad1.20x1.40mm_HandSolder, symbol Device:R
Connections:
- net +5V: now also R10.2
- net GND: now also C19.1, D4.1 (K)
- net VCC_PA_B: now also C19.2
- net at L1.2, L1.3: now also Q1.1 (B)
- net at R5.2, R6.2: now also Q1.3 (E)
- net at L2.2, L2.3: now also Q1.2 (C)
- new net: D4.2 (A), R10.1
Other:
- moved on the sheet: U1

Commit message: add mods
Parts:
- added C20: 470uF, Capacitor_SMD:C_0805_2012Metric_Pad1.18x1.45mm_HandSolder, symbol Device:C_Polarized_Small
- added J4: Conn_01x02, Jumper:SolderJumper-2_P1.3mm_Open_RoundedPad1.0x1.5mm, symbol Connector_Generic:Conn_01x02
- D1: footprint Diode_SMD:D_MiniMELF -> Diode_SMD:D_MiniMELF_Handsoldering
- D2, D3: footprint Diode_SMD:D_MiniMELF_Handsoldering -> Diode_SMD:D_MiniMELF
- Q2, Q3: footprint Package_TO_SOT_SMD:SOT-416 -> Custom:DTC114EE
Connections:
- net GND: now also C20.2
- net VCC_PA_A: now also C20.1
- net VCC_PA_B: now also J4.1 (Pin_1); no longer C4.2, L3.1
- new net: C4.2, J4.2 (Pin_2), L3.1
Other:
- moved on the sheet: J2
Changed lines of the file:
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@@
   (junction (at 43.18 78.74) (diameter 0) (color 0 0 0 0)
   )
+  (junction (at 118.11 38.1) (diameter 0) (color 0 0 0 0)
+  )
   (junction (at 154.94 85.09) (diameter 0) (color 0 0 0 0)
   )
@@
     (stroke (width 0) (type default) (color 0 0 0 0))
   )
+  (wire (pts (xy 111.76 38.1) (xy 118.11 38.1))
+    (stroke (width 0) (type default) (color 0 0 0 0))
+  )
   (wire (pts (xy 78.74 104.14) (xy 81.28 104.14))
     (stroke (width 0) (type default) (color 0 0 0 0))
@@
     (stroke (width 0) (type default) (color 0 0 0 0))
   )
-  (wire (pts (xy 121.92 38.1) (xy 127 38.1))
+  (wire (pts (xy 118.11 38.1) (xy 127 38.1))
     (stroke (width 0) (type default) (color 0 0 0 0))
   )
@@
     )
   )
-  (global_label "VCC_PA_B" (shape input) (at 124.46 57.15 180) (fields_autoplaced)
+  (global_label "VCC_PA_B" (shape input) (at 121.92 57.15 180) (fields_autoplaced)
     (effects (font (size 1.27 1.27)) (justify right))
-    (property "Intersheet References" "${INTERSHEET_REFS}" (id 0) (at 112.8545 57.0706 0)
+    (property "Intersheet References" "${INTERSHEET_REFS}" (id 0) (at 110.3145 57.0706 0)
       (effects (font (size 1.27 1.27)) (justify right) hide)
     )
@@
       (effects (font (size 1.27 1.27)) hide)
     )
-    (property "Value" "GND" (id 1) (at 137.16 50.8 0))
+    (property "Value" "GND" (id 1) (at 139.7 49.53 0))
     (property "Footprint" "" (id 2) (at 137.16 45.72 0)
       (effects (font (size 1.27 1.27)) hide)
@@
       (effects (font (size 1.27 1.27)) hide)
     )
+  )
+  (symbol (lib_id "Device:C_Polarized_Small") (at 118.11 40.64 0) (unit 1)
+    (in_bom yes) (on_board yes)
+    (property "Reference" "C20" (id 0) (at 120.269 39.2592 0)
+      (effects (font (size 1.27 1.27)) (justify left))
+    )
+    (property "Value" "470uF" (id 1) (at 109.22 43.18 0)
+      (effects (font (size 1.27 1.27)) (justify left))
+    )
+    (property "Footprint" "Capacitor_SMD:C_0805_2012Metric_Pad1.18x1.45mm_HandSolder" (id 2) (at 118.11 40.64 0)
+      (effects (font (size 1.27 1.27)) hide)
+    )
+    (property "Datasheet" "~" (id 3) (at 118.11 40.64 0)
+      (effects (font (size 1.27 1.27)) hide)
+    )
+    (pin "1")
+    (pin "2")
   )
   (symbol (lib_id "Mechanical:MountingHole") (at 31.75 190.5 0) (unit 1)
@@
       (effects (font (size 1.27 1.27)) (justify right))
     )
-    (property "Footprint" "Diode_SMD:D_MiniMELF" (id 2) (at 129.54 107.95 0)
+    (property "Footprint" "Diode_SMD:D_MiniMELF_Handsoldering" (id 2) (at 129.54 107.95 0)
       (effects (font (size 1.27 1.27)) hide)
     )
@@
       (effects (font (size 1.27 1.27)) hide)
     )
-    (property "Value" "GND" (id 1) (at 127 50.8 0))
+    (property "Value" "GND" (id 1) (at 128.27 49.53 0))
     (property "Footprint" "" (id 2) (at 127 45.72 0)
       (effects (font (size 1.27 1.27)) hide)
@@
       (effects (font (size 1.27 1.27)) (justify left))
     )
-    (property "Footprint" "Package_TO_SOT_SMD:SOT-416" (id 2) (at 113.03 144.78 0)
+    (property "Footprint" "Custom:DTC114EE" (id 2) (at 113.03 144.78 0)
       (effects (font (size 1.27 1.27)) (justify left) hide)
     )
@@
       (effects (font (size 1.27 1.27)) (justify right))
     )
-    (property "Footprint" "Diode_SMD:D_MiniMELF_Handsoldering" (id 2) (at 74.93 132.08 0)
+    (property "Footprint" "Diode_SMD:D_MiniMELF" (id 2) (at 74.93 132.08 0)
       (effects (font (size 1.27 1.27)) hide)
     )
@@
     (pin "2")
   )
+  (symbol (lib_id "power:GND") (at 118.11 43.18 0) (unit 1)
+    (in_bom yes) (on_board yes)
+    (property "Reference" "#PWR0103" (id 0) (at 118.11 49.53 0)
+      (effects (font (size 1.27 1.27)) hide)
+    )
+    (property "Value" "GND" (id 1) (at 119.38 46.99 0))
+    (property "Footprint" "" (id 2) (at 118.11 43.18 0)
+      (effects (font (size 1.27 1.27)) hide)
+    )
+    (property "Datasheet" "" (id 3) (at 118.11 43.18 0)
+      (effects (font (size 1.27 1.27)) hide)
+    )
+    (pin "1")
+  )
   (symbol (lib_id "Device:C") (at 81.28 107.95 180) (unit 1)
     (in_bom yes) (on_board yes)
@@
     (pin "2")
   )
+  (symbol (lib_id "Connector_Generic:Conn_01x02") (at 121.92 52.07 90) (unit 1)
+    (in_bom yes) (on_board yes)
+    (property "Reference" "J4" (id 0) (at 118.11 50.8 90)
+      (effects (font (size 1.27 1.27)) (justify right))
+    )
+    (property "Value" "Conn_01x02" (id 1) (at 107.95 53.34 90)
+      (effects (font (size 1.27 1.27)) (justify right))
+    )
+    (property "Footprint" "Jumper:SolderJumper-2_P1.3mm_Open_RoundedPad1.0x1.5mm" (id 2) (at 121.92 52.07 0)
+      (effects (font (size 1.27 1.27)) hide)
+    )
+    (property "Datasheet" "~" (id 3) (at 121.92 52.07 0)
+      (effects (font (size 1.27 1.27)) hide)
+    )
+    (pin "1")
+    (pin "2")
+  )
   (symbol (lib_id "Device:C") (at 205.74 77.47 0) (unit 1)
     (in_bom yes) (on_board yes) (fields_autoplaced)
@@
       (effects (font (size 1.27 1.27)) (justify right))
     )
-    (property "Footprint" "Diode_SMD:D_MiniMELF_Handsoldering" (id 2) (at 147.32 132.08 0)
+    (property "Footprint" "Diode_SMD:D_MiniMELF" (id 2) (at 147.32 132.08 0)
       (effects (font (size 1.27 1.27)) hide)
     )
@@
     (pin "4")
   )
-  (symbol (lib_id "Connector_Generic:Conn_01x01") (at 116.84 38.1 180) (unit 1)
-    (in_bom yes) (on_board yes) (fields_autoplaced)
-    (property "Reference" "J2" (id 0) (at 116.84 33.1302 0))
-    (property "Value" "Conn_01x01" (id 1) (at 116.84 35.6671 0))
-    (property "Footprint" "Connector_PinHeader_2.54mm:PinHeader_1x01_P2.54mm_Vertical" (id 2) (at 116.84 38.1 0)
-      (effects (font (size 1.27 1.27)) hide)
-    )
-    (property "Datasheet" "~" (id 3) (at 116.84 38.1 0)
+  (symbol (lib_id "Connector_Generic:Conn_01x01") (at 106.68 38.1 180) (unit 1)
+    (in_bom yes) (on_board yes) (fields_autoplaced)
+    (property "Reference" "J2" (id 0) (at 106.68 33.1302 0))
+    (property "Value" "Conn_01x01" (id 1) (at 106.68 35.6671 0))
+    (property "Footprint" "Connector_PinHeader_2.54mm:PinHeader_1x01_P2.54mm_Vertical" (id 2) (at 106.68 38.1 0)
+      (effects (font (size 1.27 1.27)) hide)
+    )
+    (property "Datasheet" "~" (id 3) (at 106.68 38.1 0)
       (effects (font (size 1.27 1.27)) hide)
     )
@@
       (effects (font (size 1.27 1.27)) (justify left))
     )
-    (property "Footprint" "Package_TO_SOT_SMD:SOT-416" (id 2) (at 40.64 144.78 0)
+    (property "Footprint" "Custom:DTC114EE" (id 2) (at 40.64 144.78 0)
       (effects (font (size 1.27 1.27)) (justify left) hide)
     )
@@
       (reference "#PWR0102") (unit 1) (value "GND") (footprint "")
     )
+    (path "/a6186f88-9222-4049-8f42-55d3263e8f58"
+      (reference "#PWR0103") (unit 1) (value "GND") (footprint "")
+    )
     (path "/a07aee06-7b4f-4e8a-be32-9aa961cff1b6"
       (reference "C1") (unit 1) (value "100n") (footprint "Capacitor_SMD:C_0805_2012Metric_Pad1.18x1.45mm_HandSolder")
@@
       (reference "C19") (unit 1) (value "100n") (footprint "Capacitor_SMD:C_0805_2012Metric_Pad1.18x1.45mm_HandSolder")
     )
+    (path "/0daecdde-c7bb-438a-af7a-81cb9557ce6b"
+      (reference "C20") (unit 1) (value "470uF") (footprint "Capacitor_SMD:C_0805_2012Metric_Pad1.18x1.45mm_HandSolder")
+    )
     (path "/30b89d76-f430-4e58-b88d-70e26cfa2473"
-      (reference "D1") (unit 1) (value "1N4007") (footprint "Diode_SMD:D_MiniMELF")
+      (reference "D1") (unit 1) (value "1N4007") (footprint "Diode_SMD:D_MiniMELF_Handsoldering")
     )
     (path "/975df7ba-4f84-400e-8112-520cb6d58c09"
-      (reference "D2") (unit 1) (value "LL4148") (footprint "Diode_SMD:D_MiniMELF_Handsoldering")
+      (reference "D2") (unit 1) (value "LL4148") (footprint "Diode_SMD:D_MiniMELF")
     )
     (path "/d233d83d-fe57-42d0-9c98-4cb5d42655dc"
-      (reference "D3") (unit 1) (value "LL4148") (footprint "Diode_SMD:D_MiniMELF_Handsoldering")
+      (reference "D3") (unit 1) (value "LL4148") (footprint "Diode_SMD:D_MiniMELF")
     )
     (path "/ebc05d4e-ad2b-4267-bddb-704aafe43beb"
@@
       (reference "J3") (unit 1) (value "Conn_01x04") (footprint "Connector_PinHeader_2.54mm:PinHeader_1x04_P2.54mm_Vertical")
     )
+    (path "/b0e1ba30-3d47-4cfc-b463-17bf7eb4384b"
+      (reference "J4") (unit 1) (value "Conn_01x02") (footprint "Jumper:SolderJumper-2_P1.3mm_Open_RoundedPad1.0x1.5mm")
+    )
     (path "/bc884ff4-0e5a-45a6-bab1-79666f59a4e8"
       (reference "J5") (unit 1) (value "Conn_01x02") (footprint "Connector_PinHeader_1.27mm:PinHeader_1x02_P1.27mm_Vertical")
@@
     )
     (path "/eb910e09-5531-4f2d-9efe-ba20f3f591a6"
-      (reference "Q2") (unit 1) (value "DTC114EE") (footprint "Package_TO_SOT_SMD:SOT-416")
+      (reference "Q2") (unit 1) (value "DTC114EE") (footprint "Custom:DTC114EE")
     )
     (path "/66230ffb-f604-4fd2-8b8b-b28ff7b4be7f"
-      (reference "Q3") (unit 1) (value "DTC114EE") (footprint "Package_TO_SOT_SMD:SOT-416")
+      (reference "Q3") (unit 1) (value "DTC114EE") (footprint "Custom:DTC114EE")
     )
     (path "/b9b1b8c2-204f-4748-bdd3-32e2c53aed97"

Commit message: add mods
Connections:
- net VCC_PA_B: now also C4.2
- net at J4.2 (Pin_2), L3.1: no longer C4.2
Other:
- moved on the sheet: C4
Changed lines of the file:
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@@
   (junction (at 142.24 78.74) (diameter 0) (color 0 0 0 0)
   )
-  (junction (at 134.62 57.15) (diameter 0) (color 0 0 0 0)
-  )
   (junction (at 194.31 73.66) (diameter 0) (color 0 0 0 0)
   )
@@
     (stroke (width 0) (type default) (color 0 0 0 0))
   )
-  (wire (pts (xy 124.46 57.15) (xy 134.62 57.15))
+  (wire (pts (xy 124.46 57.15) (xy 138.43 57.15))
     (stroke (width 0) (type default) (color 0 0 0 0))
   )
@@
   )
   (wire (pts (xy 74.93 78.74) (xy 80.01 78.74))
-    (stroke (width 0) (type default) (color 0 0 0 0))
-  )
-  (wire (pts (xy 134.62 57.15) (xy 138.43 57.15))
     (stroke (width 0) (type default) (color 0 0 0 0))
   )
@@
     (pin "2")
   )
-  (symbol (lib_id "Device:C") (at 134.62 60.96 180) (unit 1)
-    (in_bom yes) (on_board yes) (fields_autoplaced)
-    (property "Reference" "C4" (id 0) (at 137.541 60.1253 0)
-      (effects (font (size 1.27 1.27)) (justify right))
-    )
-    (property "Value" "10n" (id 1) (at 137.541 62.6622 0)
-      (effects (font (size 1.27 1.27)) (justify right))
-    )
-    (property "Footprint" "Capacitor_SMD:C_0805_2012Metric_Pad1.18x1.45mm_HandSolder" (id 2) (at 133.6548 57.15 0)
-      (effects (font (size 1.27 1.27)) hide)
-    )
-    (property "Datasheet" "~" (id 3) (at 134.62 60.96 0)
+  (symbol (lib_id "Device:C") (at 121.92 60.96 180) (unit 1)
+    (in_bom yes) (on_board yes) (fields_autoplaced)
+    (property "Reference" "C4" (id 0) (at 124.841 60.1253 0)
+      (effects (font (size 1.27 1.27)) (justify right))
+    )
+    (property "Value" "10n" (id 1) (at 124.841 62.6622 0)
+      (effects (font (size 1.27 1.27)) (justify right))
+    )
+    (property "Footprint" "Capacitor_SMD:C_0805_2012Metric_Pad1.18x1.45mm_HandSolder" (id 2) (at 120.9548 57.15 0)
+      (effects (font (size 1.27 1.27)) hide)
+    )
+    (property "Datasheet" "~" (id 3) (at 121.92 60.96 0)
       (effects (font (size 1.27 1.27)) hide)
     )
@@
     (pin "2")
   )
-  (symbol (lib_id "power:GND") (at 134.62 64.77 0) (unit 1)
-    (in_bom yes) (on_board yes) (fields_autoplaced)
-    (property "Reference" "#PWR06" (id 0) (at 134.62 71.12 0)
-      (effects (font (size 1.27 1.27)) hide)
-    )
-    (property "Value" "GND" (id 1) (at 134.62 69.3325 0))
-    (property "Footprint" "" (id 2) (at 134.62 64.77 0)
-      (effects (font (size 1.27 1.27)) hide)
-    )
-    (property "Datasheet" "" (id 3) (at 134.62 64.77 0)
-      (effects (font (size 1.27 1.27)) hide)
-    )
+  (symbol (lib_id "power:GND") (at 121.92 64.77 0) (unit 1)
+    (in_bom yes) (on_board yes) (fields_autoplaced)
+    (property "Reference" "#PWR06" (id 0) (at 121.92 71.12 0)
+      (effects (font (size 1.27 1.27)) hide)
+    )
+    (property "Value" "GND" (id 1) (at 121.92 69.3325 0))
+    (property "Footprint" "" (id 2) (at 121.92 64.77 0)
+      (effects (font (size 1.27 1.27)) hide)
+    )
+    (property "Datasheet" "" (id 3) (at 121.92 64.77 0)
+      (effects (font (size 1.27 1.27)) hide)
+    )

Commit message: add mods
Parts:
- C6: footprint Capacitor_SMD:C_0805_2012Metric_Pad1.18x1.45mm_HandSolder -> Capacitor_SMD:C_0402_1005Metric
- R7, R8: value 43 -> 220
Connections:
- net +5V: no longer R7.1, R8.1
- net VCC_PA_A: now also R7.1, R8.1
Changed lines of the file:
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@@
+    )
+  )
+  (global_label "VCC_PA_A" (shape input) (at 162.56 139.7 0) (fields_autoplaced)
+    (effects (font (size 1.27 1.27)) (justify left))
+    (property "Intersheet References" "${INTERSHEET_REFS}" (id 0) (at 173.9841 139.6206 0)
+      (effects (font (size 1.27 1.27)) (justify left) hide)
     )
   )
@@
     (property "Intersheet References" "${INTERSHEET_REFS}" (id 0) (at 32.1793 79.9306 0)
       (effects (font (size 1.27 1.27)) (justify right) hide)
+    )
+  )
+  (global_label "VCC_PA_A" (shape input) (at 90.17 139.7 0) (fields_autoplaced)
+    (effects (font (size 1.27 1.27)) (justify left))
+    (property "Intersheet References" "${INTERSHEET_REFS}" (id 0) (at 101.5941 139.6206 0)
+      (effects (font (size 1.27 1.27)) (justify left) hide)
     )
   )
@@
       (effects (font (size 1.27 1.27)) (justify right))
     )
-    (property "Footprint" "Capacitor_SMD:C_0805_2012Metric_Pad1.18x1.45mm_HandSolder" (id 2) (at 136.1948 38.1 0)
+    (property "Footprint" "Capacitor_SMD:C_0402_1005Metric" (id 2) (at 136.1948 38.1 0)
       (effects (font (size 1.27 1.27)) hide)
     )
@@
     (pin "1")
   )
-  (symbol (lib_id "power:+5V") (at 162.56 139.7 0) (unit 1)
-    (in_bom yes) (on_board yes) (fields_autoplaced)
-    (property "Reference" "#PWR032" (id 0) (at 162.56 143.51 0)
-      (effects (font (size 1.27 1.27)) hide)
-    )
-    (property "Value" "+5V" (id 1) (at 162.56 136.0955 0))
-    (property "Footprint" "" (id 2) (at 162.56 139.7 0)
-      (effects (font (size 1.27 1.27)) hide)
-    )
-    (property "Datasheet" "" (id 3) (at 162.56 139.7 0)
-      (effects (font (size 1.27 1.27)) hide)
-    )
-    (pin "1")
-  )
   (symbol (lib_id "power:+12V") (at 81.28 22.86 0) (unit 1)
     (in_bom yes) (on_board yes) (fields_autoplaced)
@@
   (symbol (lib_id "Device:R") (at 158.75 139.7 270) (unit 1)
     (in_bom yes) (on_board yes) (fields_autoplaced)
-    (property "Reference" "R8" (id 0) (at 158.75 134.7175 90))
-    (property "Value" "43" (id 1) (at 158.75 137.4926 90))
+    (property "Reference" "R8" (id 0) (at 158.75 134.9842 90))
+    (property "Value" "220" (id 1) (at 158.75 137.5211 90))
     (property "Footprint" "Resistor_SMD:R_0805_2012Metric_Pad1.20x1.40mm_HandSolder" (id 2) (at 158.75 137.922 90)
       (effects (font (size 1.27 1.27)) hide)
@@
   (symbol (lib_id "Device:R") (at 86.36 139.7 270) (unit 1)
     (in_bom yes) (on_board yes) (fields_autoplaced)
-    (property "Reference" "R7" (id 0) (at 86.36 134.7175 90))
-    (property "Value" "43" (id 1) (at 86.36 137.4926 90))
+    (property "Reference" "R7" (id 0) (at 86.36 134.9842 90))
+    (property "Value" "220" (id 1) (at 86.36 137.5211 90))
     (property "Footprint" "Resistor_SMD:R_0805_2012Metric_Pad1.20x1.40mm_HandSolder" (id 2) (at 86.36 137.922 90)
       (effects (font (size 1.27 1.27)) hide)
@@
     )
     (property "Datasheet" "" (id 3) (at 149.86 64.77 0)
-      (effects (font (size 1.27 1.27)) hide)
-    )
-    (pin "1")
-  )
-  (symbol (lib_id "power:+5V") (at 90.17 139.7 0) (unit 1)
-    (in_bom yes) (on_board yes) (fields_autoplaced)
-    (property "Reference" "#PWR025" (id 0) (at 90.17 143.51 0)
-      (effects (font (size 1.27 1.27)) hide)
-    )
-    (property "Value" "+5V" (id 1) (at 90.17 136.0955 0))
-    (property "Footprint" "" (id 2) (at 90.17 139.7 0)
-      (effects (font (size 1.27 1.27)) hide)
-    )
-    (property "Datasheet" "" (id 3) (at 90.17 139.7 0)
       (effects (font (size 1.27 1.27)) hide)
     )
@@
       (reference "#PWR024") (unit 1) (value "GND") (footprint "")
     )
-    (path "/edd4ebbb-3fed-45d9-98a0-dad956c73fd4"
-      (reference "#PWR025") (unit 1) (value "+5V") (footprint "")
-    )
     (path "/28376e63-cc44-4f2a-9460-fffbe1f00dcd"
       (reference "#PWR026") (unit 1) (value "GND") (footprint "")
@@
       (reference "#PWR031") (unit 1) (value "GND") (footprint "")
     )
-    (path "/4b7ff3d4-0570-4dfc-9955-346d5313d005"
-      (reference "#PWR032") (unit 1) (value "+5V") (footprint "")
-    )
     (path "/b7ef7806-35d8-4f7e-af7c-742af124ae51"
       (reference "#PWR033") (unit 1) (value "GND") (footprint "")
@@
     )
     (path "/471d61c9-4065-4040-bd13-0062719798cf"
-      (reference "C6") (unit 1) (value "100n") (footprint "Capacitor_SMD:C_0805_2012Metric_Pad1.18x1.45mm_HandSolder")
+      (reference "C6") (unit 1) (value "100n") (footprint "Capacitor_SMD:C_0402_1005Metric")
     )
     (path "/aadefebb-9f42-404e-806e-604ecd1a3e28"
@@
     )
     (path "/af638b05-127a-436b-9d31-94d5e9402d7e"
-      (reference "R7") (unit 1) (value "43") (footprint "Resistor_SMD:R_0805_2012Metric_Pad1.20x1.40mm_HandSolder")
+      (reference "R7") (unit 1) (value "220") (footprint "Resistor_SMD:R_0805_2012Metric_Pad1.20x1.40mm_HandSolder")
     )
     (path "/7caabdfa-ba09-4df8-b399-399265c09ef0"
-      (reference "R8") (unit 1) (value "43") (footprint "Resistor_SMD:R_0805_2012Metric_Pad1.20x1.40mm_HandSolder")
+      (reference "R8") (unit 1) (value "220") (footprint "Resistor_SMD:R_0805_2012Metric_Pad1.20x1.40mm_HandSolder")
     )
     (path "/9d252c01-363c-4fe0-b1b9-1592efd383f0"

Commit message: add mods
Parts:
- C14: value 220p -> 240p
- C18: value 100n -> 10n
- D4: value LED -> LED 2mA
- L1: value TRANSF1 -> Bifilar 6tr
- L2: value TRANSF1 -> TRANSF 2tr:3tr BN43-202
- L4, L5: value T50-6 8tr -> T37-6 8tr
- Q1: value 2SC1969 -> IRF530; footprint Package_TO_SOT_THT:TO-220-3_Horizontal_TabDown -> Package_TO_SOT_THT:TO-220-3_Vertical; symbol Transistor_BJT:2SD1047 -> Transistor_FET:IRF540N
- R10: value 420 -> 1.6k
- R4: value 27 -> 500
- R5, R6: value 1 -> 0.5
Other:
- note added: "10w 10m band Power Amplifier for uSDX mOnO. :)"
- note added: "Do not install the plate on the TRX. Put the +12 on J2 and GND on the GND of the antenna output pinheader. Put a wire on PTT. Activate when measuring. Activate the PTT and measure the voltage on pin 1 Gate of the IRF530 and adjust RV1 to have the minimum, around 2.5v. Stop the PTT then put an amp on J4. Activate the PTT and increase the bias with RV1 until you measure 15mA to 20mA. Stop the PTT a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"
- note added: "Dont place D1, it's only for old PNP purpose"
- note added: "L1 : 6tr twisted bifilar 0,35mm on FT37-43 L2 : 2tr 1 to 3, 3tr 2 to 4 twisted bifilar 0,85mm on FT37-43 BN43-202 Last turn of L2 is untwisted."
- note added: "L4 and L5 T37-6 9tr 0,85mm"
- note added: "R5 and R6, place 2x 0.5ohm 250mw or 4x 1ohm 125mw"
- note added: "Shunt attenuator if you whant."
- note added: "Shunt attenuator if you what. So replace R2 with a wire, remove R1 and R3."
- note added: "https://www.qsl.net/va3iul/Homebrew_RF_Circuit_Design_Ideas/10m_10W_SSB_PA_NZ5G.gif http://lpistor.chez-alice.fr/pa8w.htm https://electronicprojectsforfun.files.wordpress.com/2017/09/mediumpowerrfamplifierschematics.png"
- note added: "mOnO Mod: solder a wire on the back of the main board power connector and J2 to bring the +12. Solder a wire on pin 8 of U3 (74ACT00) and PTT on J5."
- note removed: "L1 : 8 spires bifilaires torsadées fil émaillé 0,5mm sur tore FT37-43 L2 : 12 spires bifilaires torsadées fil émaillé 0,5mm sur tore FT37-43"
- note removed: "https://www.qsl.net/va3iul/Homebrew_RF_Circuit_Design_Ideas/10m_10W_SSB_PA_NZ5G.gif http://lpistor.chez-alice.fr/pa8w.htm"
- moved on the sheet: J1, J3

Commit message: add mods and simulation files
Parts:
- D2, D3: value LL4148 -> BZV55-C3V3; symbol Device:D -> Device:D_Zener
- L3: value VK200 (bobinée entièrement) -> VK200 (fully wound)
Other:
- note added: "*"
- note added: "C4 you can add a 100uF in parallel"
- note added: "Do not install the plate on the TRX. Put the +12 on J2 and GND on the GND of the antenna output pinheader. Put a wire on PTT. +12v Activation when measuring. Activate the PTT and measure the voltage on pin 1 Gate of the IRF530 and adjust RV1 to have the minimum, around 2.5v. Stop the PTT then put an amp on J4. Activate the PTT and increase the bias with RV1 until you measure 15mA to 20mA. Stop th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"
- note added: "R5 and R6, place 2x 0.5ohm 250mw or 4x 1ohm 125mw You can add a 100nF capacitor in parallel"
- note removed: "Do not install the plate on the TRX. Put the +12 on J2 and GND on the GND of the antenna output pinheader. Put a wire on PTT. Activate when measuring. Activate the PTT and measure the voltage on pin 1 Gate of the IRF530 and adjust RV1 to have the minimum, around 2.5v. Stop the PTT then put an amp on J4. Activate the PTT and increase the bias with RV1 until you measure 15mA to 20mA. Stop the PTT a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"
- note removed: "R5 and R6, place 2x 0.5ohm 250mw or 4x 1ohm 125mw"
- moved on the sheet: C1, C10, C11, C12, C13, C14, C15, C16, C17, C18, C19, C2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
